File: electronic schematic/Netzteil.sch (EAGLE design)
At the start: 27 parts, among them IC1 TPS54331, IC2 INA168, U1 MCP41XXX

Commit message: new layout and schematic
Parts:
- removed D_VOLTAGE: 1N5817-B, diode:1N5817-B
- removed R_OUT: 10k?, rcl:R-EU_0204/7
- removed U1: MCP41XXX, SparkFun-AnalogIC:MCP41XXX
- added IC3: LT1257N, linear-technology:LT1257N
- added IC4: LM358N, linear:LM358N
- added RD1, RD3: 10k, rcl:R-EU_0309/12
- added RD2, RO1: 100k, resistor:R-TRIMM64Y
- added RD4: 47k, rcl:R-EU_0309/12
- added RV: 390k, rcl:R-EU_0309/12
- D_OUT: value SB120 -> SB320; device diode:SB120 -> diode:SB320
- RO2: value (none) -> 10k; device rcl:R-EU_0204/7 -> rcl:R-EU_0309/12
- R_COMP: device rcl:R-EU_0204/7 -> rcl:R-EU_0309/12
- R_SHUNT: device rcl:R-EU_0204/7 -> rcl:R-EU_0817/22
- renumbered R_AMPERE to R_A, R_VOLTAGE to R_V
Connections:
- removed net N$18: SV2.9, U1.CS
- removed net N$19: SV2.7, U1.SCK
- removed net N$20: SV2.5, U1.DI
- removed net VSS: CI1.+, CI2.+, DC1.VIN, H3.P$1, IC1.VIN
- new net +24V: CI1.+, CI2.+, DC1.VIN, H3.P$1, IC1.VIN, IC4P.V+
- new net CS: IC3.!LOAD, SV2.5
- new net MOSI: IC3.DIN, SV2.9
- new net N$11: IC1.VSENSE, IC4A.OUT, RD2.E, RD2.S
- new net N$12: IC3.VOUT, IC4B.+IN
- new net N$13: IC4B.-IN, RO1.E, RO1.S, RO2.2
- new net N$14: IC4A.-IN, RD1.2, RD2.A
- new net N$16: IC4A.+IN, RD3.2, RD4.2
- new net SCK: IC3.CLK, SV2.7
- net +5V: now also IC3.VCC; no longer D_VOLTAGE.C, IC1.EN, U1.VCC
- net GND: now also IC3.GND, IC4P.V-, RD4.1, RO2.1; no longer U1.A, U1.GND, U1.W
- net N$10: no longer D_VOLTAGE.A
- net N$4: now also IC4B.OUT, RD1.1, RO1.A; no longer IC1.VSENSE, R_OUT.1, U1.B
- net N$6: now also RD3.1, RV.1; no longer RO2.1, R_OUT.2
- net N$9: now also RV.2; no longer RO2.2
Other:
- moved on the sheet: C5V1, C5V2, CSS, C_COMP, C_COMPR, C_OUT, D_OUT, RO2, R_COMP
