File: electronic schematic/Steuerung.sch (EAGLE design)
At the start: 22 parts, among them IC3 MEGA16-P, SW1 EC12E_SW, U2 LCD-16X2SILK

Commit message: new layout and schematic
Parts:
- removed JP3: (no value), pinhead:PINHD-1X3
- removed L2: (no value), rcl:L-EUPIS2816
- removed RLCD1, RLCD2, RLCD3: (no value), rcl:R-EU_0204/7
- removed S1: (no value), SparkFun-Electromechanical:SWITCH-SPDTPTH
- added CKTRST: 100n, resistor:C-EUC1206K
- added R4: 100k, resistor:R-EU_R1206W
- added R5, R6: 4.7k, resistor:R-EU_R1206W
- added R_RESET: (no value), rcl:R-EU_R1206W
- C5V3: value (none) -> 1n; device eagle-ltspice:CC1206 -> resistor:C-EUC1206K
- CX1, CX2: value (none) -> 18p
- D2, D3: value BAT60J -> ZPD; device diode:BAT60J -> diode:ZPD
- JP1: device pinhead:PINHD-1X8 -> pinhead:PINHD-1X9
- RD+, RD-, RD-V, RLCD: device rcl:R-EU_0204/7 -> rcl:R-EU_0309/12
- SV2: device con-ml:ML10 -> con-harting-ml:ML10
Connections:
- removed net N$16: RLCD.2, S1.P
- removed net N$36: JP3.2, U2.VO
- removed net N$37: IC3.AREF, IC3.AVCC, L2.2
- new net KONTRAST: CKTRST.1, R4.1, R5.1, R6.1, U2.VO
- new net N$5: IC3.RESET, R_RESET.2
- new net PWM: IC3.(OC1A)PD5, R5.2
- net +5V: now also IC3.AVCC, R4.2, RLCD.2, R_RESET.1; no longer JP3.1, L2.1, S1.O, SW1G$1.C, SW1G$2.1
- net GND: now also CKTRST.2, JP1.9, R6.2, SW1G$1.C, SW1G$2.1; no longer JP3.3, RLCD1.2, RLCD2.2, RLCD3.2, S1.S
- net N$18: now also SV2.5; no longer SV2.9
- net N$2: no longer RLCD1.1
- net N$20: now also SV2.9; no longer SV2.5
- net N$3: no longer RLCD2.1
- net N$4: no longer RLCD3.1
